File: Onboarding Project.kicad_sch (KiCad schematic)
At the start: 68 parts, among them J1 Conn_01x04_Pin, J2 Conn_01x04_Pin, J3 Conn_01x04_Pin, J4 USB_C_Receptacle_USB2.0_14P, J5 Conn_01x02_Pin, J6 Conn_01x04_Pin, J7 Conn_01x06_Pin, J8 Conn_01x08_Pin, SW1 SW_SPDT, SW2 SW_Push, SW3 SW_Push, U1 STM32F103C8T6, U2 AMS1117-3.3, U3 PAM8302AAS, Y1 16MHz

Commit message: Completed
Parts:
- removed J3: Conn_01x04_Pin, Connector_PinHeader_2.54mm:PinHeader_1x04_P2.54mm_Vertical, symbol Connector:Conn_01x04_Pin
- removed J7: Conn_01x06_Pin, Connector_PinHeader_2.54mm:PinHeader_1x06_P2.54mm_Vertical, symbol Connector:Conn_01x06_Pin
- removed J8: Conn_01x08_Pin, Connector_PinHeader_2.54mm:PinHeader_1x08_P2.54mm_Vertical, symbol Connector:Conn_01x08_Pin
- removed R4, R5: 1k5, Resistor_SMD:R_0402_1005Metric, symbol Device:R
- removed R9: 10k, Resistor_SMD:R_0402_1005Metric, symbol Device:R
- removed SW3: SW_Push, Button_Switch_THT:SW_NKK_GW12LJP, symbol Switch:SW_Push
- added H1, H2, H3, H4: MountingHole, MountingHole:MountingHole_2.2mm_M2, symbol Mechanical:MountingHole
- J4: footprint (none) -> Connector_USB:USB_C_Receptacle_HRO_TYPE-C-31-M-12
- SW1: footprint Button_Switch_THT:SW_Lever_1P2T_NKK_GW12LxH -> Button_Switch_SMD:SW_SPDT_PCM12
Connections:
- net SWPUSH: no longer U1.25 (PB12)
- net I2C2_SCL: no longer names the net of U1.21 (PB10)
- net I2C2_SDA: no longer names the net of U1.22 (PB11)
- net SPI2_CS: no longer names the net of U1.16 (PA6)
- net SPI2_MISO: no longer names the net of U1.27 (PB14)
- net SPI2_MOS1: no longer names the net of U1.28 (PB15)
- net SPI2_SCK: no longer names the net of U1.26 (PB13)
- no-connect marks 8 -> 15
Other:
- note added: "M2"
- note added: "Mounting Holes"
