File: Onboarding Project.kicad_pcb (KiCad board)
At the start: 2 copper layers, 54 x 54.8 mm, 65 parts, among them J1 Conn_01x04_Pin, J2 Conn_01x04_Pin, J4 USB_C_Receptacle_USB2.0_14P, J5 Conn_01x02_Pin, J6 Conn_01x04_Pin, SW1 SW_SPDT, SW2 SW_Push, U1 STM32F103C8T6, U2 AMS1117-3.3, U3 PAM8302AAS, Y1 16MHz

Commit message: Clearance error fixed
Routing:
- net GND: track 68.5 -> 69.9 mm
- net VBUS: track 33.1 -> 32.7 mm, vias 4 -> 3
- net +3.3V: vias 8 -> 7
